File: PDP11Hack/JPLR J11 Hack.kicad_sch (KiCad schematic)
At the start: 24 parts, among them J1 VBAT, J2 PWR, U1 74HCT04

Commit message: Last update, PCB creation ready
Parts:
- U1: footprint (none) -> Package_DIP:DIP-14_W7.62mm
Connections:
- net BUFCTL renamed BUFCTL_hier
- net ~{BUFCTL} renamed ~{BUFCTL_hier}
Other:
- moved on the sheet: U1A
Changed lines of the file:
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@@
 	(wire
 		(pts
-			(xy 160.02 146.05) (xy 166.37 146.05)
-		)
-		(stroke
-			(width 0)
-			(type default)
-		)
-	)
-	(wire
-		(pts
 			(xy 394.97 220.98) (xy 383.54 220.98)
 		)
@@
 	(wire
 		(pts
-			(xy 27.94 36.83) (xy 36.83 36.83)
+			(xy 21.59 36.83) (xy 36.83 36.83)
 		)
 		(stroke
@@
 	(wire
 		(pts
+			(xy 124.46 146.05) (xy 129.54 146.05)
+		)
+		(stroke
+			(width 0)
+			(type default)
+		)
+	)
+	(wire
+		(pts
 			(xy 260.35 64.77) (xy 262.89 64.77)
 		)
@@
 	(wire
 		(pts
-			(xy 212.09 41.91) (xy 218.44 41.91)
+			(xy 207.01 41.91) (xy 218.44 41.91)
 		)
 		(stroke
@@
 	(wire
 		(pts
-			(xy 135.89 146.05) (xy 144.78 146.05)
-		)
-		(stroke
-			(width 0)
-			(type default)
-		)
-	)
-	(wire
-		(pts
 			(xy 214.63 120.65) (xy 218.44 120.65)
 		)
@@
 	(wire
 		(pts
-			(xy 158.75 140.97) (xy 166.37 140.97)
+			(xy 149.86 140.97) (xy 166.37 140.97)
 		)
 		(stroke
@@
 	(wire
 		(pts
-			(xy 158.75 38.1) (xy 166.37 38.1)
+			(xy 153.67 38.1) (xy 166.37 38.1)
 		)
 		(stroke
@@
 	(wire
 		(pts
-			(xy 307.34 52.07) (xy 309.88 52.07)
+			(xy 144.78 146.05) (xy 166.37 146.05)
+		)
+		(stroke
+			(width 0)
+			(type default)
+		)
+	)
+	(wire
+		(pts
+			(xy 307.34 66.04) (xy 309.88 66.04)
 		)
 		(stroke
@@
 		)
 	)
-	(label "~{BUFCTL}"
-		(at 158.75 140.97 0)
+	(label "~{BUFCTL_hier}"
+		(at 149.86 140.97 0)
 		(effects
 			(font
@@
 		)
 	)
-	(label "~{WEL}"
+	(label "~{WEL_hier}"
 		(at 255.27 41.91 0)
 		(effects
@@
 		)
 	)
-	(label "~{BUFCTL}"
+	(label "~{BUFCTL_hier}"
 		(at 252.73 105.41 0)
 		(effects
@@
 	)
 	(label "~{SCTL}"
-		(at 135.89 146.05 180)
+		(at 124.46 146.05 180)
 		(effects
 			(font
@@
 		)
 	)
-	(label "~{WEU}"
+	(label "~{WEU_hier}"
 		(at 255.27 45.72 0)
 		(effects
@@
 		)
 	)
-	(label "BUFCTL"
+	(label "BUFCTL_hier"
 		(at 158.75 135.89 0)
 		(effects
@@
 		)
 	)
-	(label "~{BUFCTL}"
+	(label "~{BUFCTL_hier}"
 		(at 130.81 129.54 0)
 		(effects
@@
 		)
 	)
-	(label "~{WEU}"
+	(label "~{WEU_hier}"
 		(at 300.99 44.45 0)
 		(effects
@@
 		)
 	)
-	(label "~{WEL}"
-		(at 212.09 41.91 0)
+	(label "~{WEL_hier}"
+		(at 207.01 41.91 0)
 		(effects
 			(font
@@
 		)
 	)
-	(label "~{WEL}"
+	(label "~{WEL_hier}"
 		(at 300.99 40.64 0)
 		(effects
@@
 		)
 	)
-	(label "~{BUFCTL}"
-		(at 307.34 52.07 180)
+	(label "~{BUFCTL_hier}"
+		(at 307.34 66.04 180)
 		(effects
 			(font
@@
 		)
 	)
-	(label "~{BUFCTL}"
-		(at 27.94 36.83 0)
+	(label "~{BUFCTL_hier}"
+		(at 21.59 36.83 0)
 		(effects
 			(font
@@
 		)
 	)
-	(label "~{BUFCTL}"
-		(at 158.75 38.1 0)
+	(label "~{BUFCTL_hier}"
+		(at 153.67 38.1 0)
 		(effects
 			(font
@@
 			)
 		)
-		(property "Footprint" ""
+		(property "Footprint" "Package_DIP:DIP-14_W7.62mm"
 			(at 280.67 259.08 0)
 			(effects
@@
 			)
 		)
-		(property "Footprint" ""
+		(property "Footprint" "Package_DIP:DIP-14_W7.62mm"
 			(at 151.13 130.81 0)
 			(effects
@@
 	(symbol
 		(lib_id "74xx:74HCT04")
-		(at 152.4 146.05 0)
+		(at 137.16 146.05 0)
 		(unit 1)
 		(exclude_from_sim no)
@@
 		(fields_autoplaced yes)
 		(property "Reference" "U1"
-			(at 152.4 137.16 0)
+			(at 137.16 137.16 0)
 			(effects
 				(font
@@
 		)
 		(property "Value" "74HCT04"
-			(at 152.4 139.7 0)
+			(at 137.16 139.7 0)
 			(effects
 				(font
@@
 			)
 		)
-		(property "Footprint" ""
-			(at 152.4 146.05 0)
+		(property "Footprint" "Package_DIP:DIP-14_W7.62mm"
+			(at 137.16 146.05 0)
 			(effects
 				(font
@@
 		)
 		(property "Datasheet" "https://assets.nexperia.com/documents/data-sheet/74HC_HCT04.pdf"
-			(at 152.4 146.05 0)
+			(at 137.16 146.05 0)
 			(effects
 				(font
@@
 		)
 		(property "Description" "Hex Inverter"
-			(at 152.4 146.05 0)
+			(at 137.16 146.05 0)
 			(effects
 				(font
@@
 		)
 		(pin "~{nBufCTL}" input
-			(at 309.88 52.07 180)
+			(at 309.88 66.04 180)
 			(effects
 				(font
