File: SYM-1_65816/SYM-1/ROMS.kicad_sch (KiCad schematic)
At the start: 72 parts, among them U10 74LS156, U11 74LS156, U20 27C64, U209 74LS40, U21 27C64, U22 CY62256-70PC, U23 CY62256-70PC, U24 74LS08, U39 74AHC04

Commit message: No Kicad errors but still unsusable
Connections:
- net higher_64K is gone; now on net Higher_64K: U24.10, U24.5
- net ~{higher_64K} renamed ~{Higher_64K}
Changed lines of the file:
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@@
 	)
 	(no_connect
-		(at 242.57 144.78)
+		(at 213.36 175.26)
 	)
 	(no_connect
-		(at 213.36 175.26)
+		(at 242.57 144.78)
 	)
 	(no_connect
@@
 	(wire
 		(pts
+			(xy 228.6 144.78) (xy 242.57 144.78)
+		)
+		(stroke
+			(width 0)
+			(type default)
+		)
+	)
+	(wire
+		(pts
 			(xy 199.39 198.12) (xy 199.39 205.74)
 		)
@@
 	(wire
 		(pts
-			(xy 228.6 144.78) (xy 242.57 144.78)
-		)
-		(stroke
-			(width 0)
-			(type default)
-		)
-	)
-	(wire
-		(pts
 			(xy 153.67 250.19) (xy 181.61 250.19)
 		)
@@
 		)
 	)
-	(hierarchical_label "~{higher_64K}"
+	(hierarchical_label "~{Higher_64K}"
 		(shape input)
 		(at 107.95 187.96 180)
@@
 		)
 	)
-	(hierarchical_label "higher_64K"
+	(hierarchical_label "Higher_64K"
 		(shape input)
 		(at 31.75 118.11 180)
