File: SYM-1_65816/SYM-1/SYM-1.kicad_sch (KiCad schematic)
At the start: 40 parts, among them U100 74HC138, U104 74AHC373, U105 74LS27, U107 74LS10, U2 74AHC04, U215 74AHC00, U3 74LS27, U39 74AHC04, U5 65816, U6 ICM7555xP, U7 74LS10, U8 74HC00, U9 74AHC04, Y1 1MHz

Commit message: No Kicad errors but still unsusable
Connections:
- net +5V: now also CR26.1 (K), P_connector1.1 (Pin_1), P_connector1.10 (Pin_10), P_connector1.3 (Pin_3), P_connector1.5 (Pin_5), U100.16 (VCC), U100.6 (E2), U104.20 (VCC), U5.8 (VCC)
- removed net VCC: CR26.1 (K), P_connector1.1 (Pin_1), P_connector1.10 (Pin_10), P_connector1.3 (Pin_3), P_connector1.5 (Pin_5), R201.2, R204.2, R205.2, R206.2, R73.2, R74.2, U100.16 (VCC), U100.6 (E2), U104.20 (VCC), U5.8 (VCC)
- new net: R201.2, R204.2, R205.2, R206.2, R73.2, R74.2
- no-connect marks 4 -> 8
Other:
- sheet Display ports: added LEDs_row_0, LEDs_row_1, LEDs_row_2, LEDs_row_3, LEDs_row_4, LEDs_row_5, LEDs_row_6; removed LEDs_Row_0, LEDs_Row_1, LEDs_Row_2, LEDs_Row_3, LEDs_Row_4, LEDs_Row_5, LEDs_Row_6
- sheet ROMS ports: added ~{Higher_64K}; removed higher_64K, ~{higher_64K}
- sheet VIAs ports: added APA[0..7], APB[0..7], U28_CA1, U28_CA2, U28_CB1, U28_CB2, U28_PA[0..7], U28_PB[0..7], U29_CA1, U29_CA2, U29_CB1, U29_CB2, U29_PA[0..7], U29_PB[0..7]; removed AA_CA1, AA_CB1, AA_conn[0..43], A_conn[0..43]
- sheet connectors ports: added AUDIN, AUD_H, AUD_L, KBD, KBD_R, PTR, PTR_R, ROW[0..3], U25_PA[0..7], U25_PB[0..7], U28_CA1, U28_CA2, U28_CB1, U28_CB2, U28_PA[0..7], U28_PB[0..7], U29_CA1, U29_CB1, U29_PA[0..7], U29_PB[0..3], {COLA COLB COLC COLD COLE COLF COLG}; removed AA_CA1, AA_CB1, AA_conn[0..43], A_conn[0..43]
- sheet keypad ports: added {COLA COLB COLC COLD COLE COLF COLG}; removed none
