File: SYM-1_65816/SYM-1/connectors.kicad_sch (KiCad schematic)
At the start: 12 parts, among them P4 POWER

Commit message: No Kicad errors but still unsusable
Connections:
- net VCC is gone; now on net +5V: A_connector1.A (+5V), E_connector1.21 (+5V)
- net GND: no longer AA_connector1.N (bn)
- net AA-10 renamed U28_PA7
- net AA-11 renamed U28_PA5
- net AA-12 renamed U28_PA3
- net AA-14 renamed U29_CB1
- net AA-15 renamed U29_PB2
- net AA-16 renamed U29_PB0
- net AA-17 renamed U29_PA6
- net AA-18 renamed U29_PA3
- net AA-19 renamed U29_PA4
- net AA-20 renamed U29_PA5
- net AA-3 renamed U28_PA1
- net AA-4 renamed U28_CA2
- net AA-5 renamed U28_CB2
- net AA-6 renamed U28_PB7
- net AA-8 renamed U28_PB3
- net AA-9 renamed U28_PB1
- net AA-C renamed U28_PA2
- net AA-D renamed U28_PA0
- net AA-H renamed U28_PB6
- net AA-J renamed U28_PB4
- net AA-K renamed U28_PB2
- net AA-L renamed U28_PB0
- net AA-M renamed U28_PA6
- net AA-N renamed U28_PB5
- net AA-P renamed U29_CA1
- net AA-S renamed U29_PB3
- net AA-T renamed U29_PB1
- net AA-U renamed U29_PA7
- net AA-V renamed U29_PA0
- net AA-W renamed U29_PA1
- net AA-X renamed U29_PA2
- net AA_CA1 renamed U28_CA1
- net AA_CB1 renamed U28_CB1
- new net U28_PA4: AA_connector1.N (bn)
Other:
- moved on the sheet: A_connector1
