File: SYM-1_65816/SYM-1/display.kicad_sch (KiCad schematic)
At the start: 35 parts, among them Q20 BC337, Q21 BC337, Q22 BC337, Q23 BC337, Q24 BC337, Q25 BC337, Q32 BC337, U31 C. ANODE, U32 C. ANODE, U33 C. ANODE, U34 C. ANODE, U35 C. ANODE, U36 C. ANODE, U37 74145

Commit message: No Kicad errors but still unsusable
Parts:
- removed U37: 74145, KIM-1_Library:DIP-16_W7.62mm_U24, symbol KIM-1_Library:74145
- added U40: 74LS145, symbol 74xx:74LS145
Connections:
- net VCC is gone; now on net +5V: Q20.1 (C), Q21.1 (C), Q22.1 (C), Q23.1 (C), Q24.1 (C), Q25.1 (C), R53.2, R54.2, R55.2, R56.2, R57.2, R58.2
- net +5V: now also U40.16 (VCC)
- net GND: now also U40.8 (GND)
- net LEDs_Enable: now also U40.12 (P3)
- net PB0_Row_1: now also U40.15 (P0)
- net PB1_Row_2: now also U40.14 (P1)
- net PB2_Row_3: now also U40.13 (P2)
- net at R51.2: now also U40.5 (Q4)
- net at R47.2: now also U40.1 (Q0)
- net at R50.2: now also U40.4 (Q3)
- net at R52.2: now also U40.6 (Q5)
- net at R48.2: now also U40.2 (Q1)
- net at Q32.2 (B), R123.1: now also U40.7 (Q6)
- net at R49.2: now also U40.3 (Q2)
- net LEDs_Row_0 renamed LEDs_row_0
- net LEDs_Row_1 renamed LEDs_row_1
- net LEDs_Row_2 renamed LEDs_row_2
- net LEDs_Row_3 renamed LEDs_row_3
- net LEDs_Row_4 renamed LEDs_row_4
- net LEDs_Row_5 renamed LEDs_row_5
- net LEDs_Row_6 renamed LEDs_row_6
