File: SYM-1_65816/SYM-1/keypad.kicad_sch (KiCad schematic)
At the start: 44 parts, among them U27 W65C22NxP, U30 74LS06, U38 74LS06, U7 74LS10, U8 74HC00, U9 74AHC04

Commit message: No Kicad errors but still unsusable
Connections:
- net VCC is gone; now on net +5V: K_connector1.1 (Pin_1), K_connector1.2 (Pin_2), K_connector1.3 (Pin_3), K_connector1.4 (Pin_4), R83.1, U27.20 (VCC)
