File: SYM-1_65816/SYM-1/ram.kicad_sch (KiCad schematic)
At the start: 25 parts, among them U1 74HC138, U12 2114, U13 2114, U14 2114, U15 2114, U16 2114, U17 2114, U18 2114, U19 2114, U2 74AHC04, U3 74LS27, U4 74HC00

Commit message: No Kicad errors but still unsusable
Connections:
- net VCC is gone; now on net +5V: U12.18 (VCC), U13.18 (VCC), U14.18 (VCC), U15.18 (VCC), U16.18 (VCC), U17.18 (VCC), U18.18 (VCC), U19.18 (VCC)
